Commit message: Replace Gazebo sim with IsaacGym; add G1 standing demo
Removes g1_gazebo (world, ros2_control position controllers, spawn
launch) and the gazebo-only urdf overlay, since we're moving simulation
to IsaacGym instead.

Adds g1_isaacgym: a standalone script (runs under the dexman_isaacgym
conda env, not colcon) that loads g1_description's URDF into IsaacGym
and stands the robot up using Unitree's own pretrained leg policy
(unitreerobotics/unitree_rl_gym's deploy/pre_train/g1/motion.pt, copied
in with attribution) run closed-loop with a zero velocity command. A
fixed-pose PD hold with no policy reliably topples the robot forward
within ~1s in this sim, hence the policy.

Also adds an optional UDP bridge (rviz_bridge.py + isaacgym_rviz.launch.py)
so RViz can mirror the live sim's joint states and pelvis pose alongside
the IsaacGym viewer window, kept as a separate ROS process from the
conda/IsaacGym one to avoid conda/system library conflicts.

Fixes an invalid `--` inside an XML comment in g1_tether.urdf that broke
strict XML parsing (needed to programmatically strip world/floating_base_joint
before handing the URDF to IsaacGym).

Co-Authored-By: Claude Sonnet 5 <noreply@anthropic.com>

File: src/g1_description/urdf/g1_tether.urdf (robot description, URDF)
Before this commit: robot g1_29dof_rev_1_0, 91 links, 90 joints
Links:
- link left_ankle_roll_link: geometry collision box size=0.15 0.08 0.03; visual mesh filename=package://g1_description/meshes/left_ankle_roll_link.STL
- link right_ankle_roll_link: geometry collision box size=0.15 0.08 0.03; visual mesh filename=package://g1_description/meshes/right_ankle_roll_link.STL

File: src/g1_description/urdf/g1_tether.urdf.xacro (robot description, xacro)
@@ -144,14 +144,15 @@
       </material>
     </visual>
-    <collision>
-      <origin xyz="0.05 0.02 -0.02" rpy="3.1415927 1.5695351 3.1415927"/>
-      <geometry>
-        <cylinder radius="0.02" length="0.15"/>
-      </geometry>
-    </collision>
-    <collision>
-      <origin xyz="0.05 -0.02 -0.02" rpy="3.1415927 1.5695351 3.1415927"/>
-      <geometry>
-        <cylinder radius="0.02" length="0.15"/>
+    <!-- A single flat sole box, not the two thin 2cm-radius cylindrical
+         "rails" this replaced: cylinder-on-ground-plane contact only
+         generates a couple of point/line contacts, which is a narrow,
+         easily-rocked support base for the ~34kg total robot weight and was
+         a major contributor to the whole model exploding/sliding on landing
+         (see g1_world.world's contact_max_correcting_vel comment). A flat
+         box gives a stable 4-corner contact patch instead. -->
+    <collision>
+      <origin xyz="0.05 0 -0.02" rpy="0 0 0"/>
+      <geometry>
+        <box size="0.15 0.08 0.03"/>
       </geometry>
     </collision>
@@ -266,14 +267,9 @@
       </material>
     </visual>
-    <collision>
-      <origin xyz="0.05 0.02 -0.02" rpy="3.1415927 1.5695351 3.1415927"/>
-      <geometry>
-        <cylinder radius="0.02" length="0.15"/>
-      </geometry>
-    </collision>
-    <collision>
-      <origin xyz="0.05 -0.02 -0.02" rpy="3.1415927 1.5695351 3.1415927"/>
-      <geometry>
-        <cylinder radius="0.02" length="0.15"/>
+    <!-- Flat sole box, see left_ankle_roll_link's collision comment. -->
+    <collision>
+      <origin xyz="0.05 0 -0.02" rpy="0 0 0"/>
+      <geometry>
+        <box size="0.15 0.08 0.03"/>
       </geometry>
     </collision>
